File: Board/BUS%2fVoltageconv.kicad_sch (KiCad schematic)
At the start: 3 parts, among them IC16 74LVC8T245SO24

Commit message: working on r3.1a
Other:
- note added: "MICROPET-V3.1A"
- note removed: "MICROPET-V3.0A"
Changed lines of the file:
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@@
 		)
 	)
-	(text "MICROPET-V3.0A"
+	(text "MICROPET-V3.1A"
 		(exclude_from_sim no)
 		(at 175.26 162.56 0)
