File: Board/CPU,RAM,ROM.kicad_sch (KiCad schematic)
At the start: 18 parts, among them IC1 RAMSOCK32TO512KSOP, IC13 RAMSOCK32TO512KSOP, IC6 74125D, IC7 74138D, U2 74LVC1G04

Commit message: working on r3.1a
Parts:
- removed IC1, IC13: RAMSOCK32TO512KSOP, micropet_v3:SOP32, symbol micropet_v3-eagle-import:RAMSOCK32TO512KSOP
- removed JS1: RENOSCXLH, micropet_v3:RENJS6, symbol micropet_v3-eagle-import:RENOSCXLH
- added IC1, IC13: 512k x8 10ns SRAM, Package_SO:TSOP-II-44_10.16x18.41mm_P0.8mm, symbol Memory_RAM:IS61C5128AL-10TLI
- added R33: 10k, Resistor_SMD:R_0805_2012Metric_Pad1.20x1.40mm_HandSolder, symbol csa_ultracpu-eagle-import:R-EU_0207/2V
- added X3: SG-8002CE, Oscillator:Oscillator_SMD_SeikoEpson_SG8002CE-4Pin_3.2x2.5mm, symbol Oscillator:SG-8002CE
- R10, R11, R9: footprint micropet_v3:0207_2V -> Resistor_SMD:R_0805_2012Metric_Pad1.20x1.40mm_HandSolder
Connections:
- net /RAMCS is gone; now on net RAMA18: U$2.59 (IO_L13N_D10_2)
- net A0: now also IC1.3 (A0)
- net A1: now also IC1.4 (A1)
- net A10: now also IC1.26 (A10)
- net A11: now also IC1.27 (A11)
- net A12: now also IC1.28 (A12)
- net A13: now also IC1.29 (A13)
- net A14: now also IC1.30 (A14)
- net A2: now also IC1.5 (A2)
- net A3: now also IC1.6 (A3)
- net A4: now also IC1.7 (A4)
- net A5: now also IC1.16 (A5)
- net A6: now also IC1.17 (A6)
- net A7: now also IC1.18 (A7)
- net A8: now also IC1.19 (A8)
- net A9: now also IC1.20 (A9)
- net D0: now also IC1.9 (I/O0)
- net D1: now also IC1.10 (I/O1)
- net D2: now also IC1.13 (I/O2)
- net D3: now also IC1.14 (I/O3)
- net D4: now also IC1.31 (I/O4)
- net D5: now also IC1.32 (I/O5)
- net D6: now also IC1.35 (I/O6)
- net D7: now also IC1.36 (I/O7)
- net FA15: now also IC1.38 (A15)
- net FA16: now also IC1.39 (A16)
- net FA17: now also IC1.40 (A17)
- net FA18: now also IC1.41 (A18)
- net GND: now also IC1.12 (GND), IC1.34 (GND), IC13.12 (GND), IC13.34 (GND), X3.2 (GND)
- net QCLK: now also X3.3 (OUT)
- net RAMA0: now also U$2.88 (IO_L42P_GCLK7_1), IC13.3 (A0); no longer U$2.51 (IO_L31P_GCLK31_D14_2)
- net RAMA1: now also U$2.87 (IO_L42N_GCLK6_TRDY1_1), IC13.4 (A1); no longer U$2.56 (IO_L30P_GCLK1_D13_2)
- net RAMA10: now also U$2.47 (IO_L48N_RDRW_B_VREF_2), IC13.26 (A10); no longer U$2.57 (IO_L14N_D12_2)
- net RAMA11: now also U$2.46 (IO_L49P_D3_2), IC13.27 (A11); no longer U$2.62 (IO_L12P_D1_MISO2_2)
- net RAMA12: now also U$2.45 (IO_L49N_D4_2), IC13.28 (A12); no longer U$2.81 (IO_L46P_1)
- net RAMA13: now also U$2.44 (IO_L62P_D5_2), IC13.29 (A13); no longer U$2.80 (IO_L46N_1)
- net RAMA14: now also U$2.43 (IO_L62N_D6_2), IC13.30 (A14); no longer U$2.83 (IO_L45P_1)
- net RAMA15: now also U$2.56 (IO_L30P_GCLK1_D13_2), IC13.38 (A15); no longer U$2.87 (IO_L42N_GCLK6_TRDY1_1)
- net RAMA16: now also U$2.57 (IO_L14N_D12_2), IC13.39 (A16); no longer U$2.85 (IO_L43P_GCLK5_1)
- net RAMA17: now also U$2.58 (IO_L14P_D11_2), IC13.40 (A17); no longer U$2.84 (IO_L43N_GCLK4_1)
- net RAMA18: now also IC13.41 (A18); no longer U$2.88 (IO_L42P_GCLK7_1)
- net RAMA2: now also U$2.85 (IO_L43P_GCLK5_1), IC13.5 (A2); no longer U$2.58 (IO_L14P_D11_2)
- net RAMA3: now also U$2.84 (IO_L43N_GCLK4_1), IC13.6 (A3); no longer IC6.3 (O), U$2.60 (IO_L13P_M1_2)
- net RAMA4: now also U$2.83 (IO_L45P_1), IC13.7 (A4); no longer U$2.61 (IO_L12N_D2_MISO3_2)
- net RAMA5: now also IC6.3 (O), U$2.60 (IO_L13P_M1_2), IC13.16 (A5); no longer U$2.66 (IO_L2N_CMPMOSI_2)
- net RAMA6: now also U$2.61 (IO_L12N_D2_MISO3_2), IC13.17 (A6); no longer U$2.75 (IO_L74P_AWAKE_1)
- net RAMA7: now also U$2.62 (IO_L12P_D1_MISO2_2), IC13.18 (A7); no longer U$2.79 (IO_L47P_1)
- net RAMA8: now also U$2.66 (IO_L2N_CMPMOSI_2), IC13.19 (A8); no longer U$2.78 (IO_L47N_1)
- net RAMA9: now also IC13.20 (A9)
- net RAMD0: now also U$2.81 (IO_L46P_1), IC13.9 (I/O0); no longer U$2.48 (IO_L48P_D7_2)
- net RAMD1: now also U$2.80 (IO_L46N_1), IC13.10 (I/O1); no longer U$2.46 (IO_L49P_D3_2)
- net RAMD2: now also U$2.79 (IO_L47P_1), IC13.13 (I/O2); no longer U$2.44 (IO_L62P_D5_2)
- net RAMD3: now also U$2.78 (IO_L47N_1), IC13.14 (I/O3); no longer U$2.43 (IO_L62N_D6_2)
- net RAMD4: now also U$2.48 (IO_L48P_D7_2), IC13.31 (I/O4); no longer U$2.45 (IO_L49N_D4_2)
- net RAMD5: now also U$2.50 (IO_L31N_GCLK30_D15_2), IC13.32 (I/O5); no longer U$2.47 (IO_L48N_RDRW_B_VREF_2)
- net RAMD6: now also U$2.51 (IO_L31P_GCLK31_D14_2), IC13.35 (I/O6); no longer U$2.50 (IO_L31N_GCLK30_D15_2)
- net RAMD7: now also IC13.36 (I/O7)
- net V33: now also IC1.11 (VDD), IC1.33 (VDD), IC13.11 (VDD), IC13.33 (VDD), R33.1, X3.4 (Vcc)
- net /RAMWE renamed /RAMCS
- net /RAMCS: now also IC13.37 (~{OE}), IC13.8 (~{CE})
- new net: R33.2, X3.1 (OE)
- new net R/-W: IC1.15 (~{WE})
- new net /FRAMSEL: IC1.37 (~{OE}), IC1.8 (~{CE})
- new net /RAMWE: IC13.15 (~{WE}), U$2.75 (IO_L74P_AWAKE_1)
Other:
- note added: "3.0B: - add pulldown on /RES during FPGA config 3.1A: - replace 5V SRAM with 3.3V SRAM in TSOP2-44 - replace clock oscillator with more common footprint - Change 33R 10kR footprints to SMD"
- note added: "MICROPET-V3.1A"
- note added: "MICROPET-V3.1A-20241230"
- note removed: "3.0B: - add pulldown on /RES during FPGA config"
- note removed: "MICROPET-V3.0B"
- note removed: "MICROPET-V3.0B-20240523"

Commit message: draft final layout mupet 3.1a
Parts:
- removed IC7: 74138D, micropet_v3:SO16, symbol micropet_v3-eagle-import:74138D
- added C72, C73, C74: 0.1u, Capacitor_SMD:C_0603_1608Metric, symbol Device:C_Small
Connections:
- net /BE_OUT is gone; now on net /FRAMSEL: U$2.132 (IO_L35P_GCLK17_0)
- net BE_IN is gone; now on net IGOUT: U$2.118 (IO_L63N_SCP6_0)
- net C2PHI2 is gone; now on net SPI_NSEL5: U$2.104 (IO_L1N_VREF_1)
- net C8PHI2 is gone; now on net SPI_NFLASH: U$2.102 (IO_L32P_1)
- net SPISELA is gone; now on net /FPGABOOT: U$2.38 (IO_L65N_CSO_B_2)
- net SYNC is gone; now on net ROUT: U$2.121 (IO_L62P_0)
- net /FRAMSEL: no longer U$2.120 (IO_L62N_VREF_0)
- net /LDAC: now also U$2.126 (IO_L36N_GCLK14_0); no longer U$2.138 (IO_L4P_0)
- net /RES: now also U$2.98 (IO_L34P_1); no longer U$2.117 (IO_L64P_SCP5_0)
- net /SEL1: now also U$2.93 (IO_L41P_GCLK9_IRDY1_1); no longer U$2.134 (IO_L34P_GCLK19_0)
- net /SEL2: now also U$2.92 (IO_L41N_GCLK8_1); no longer U$2.115 (IO_L65P_SCP3_0)
- net /SEL4: now also U$2.88 (IO_L42P_GCLK7_1); no longer U$2.111 (IO_L66N_SCP0_0)
- net A12: now also U$2.138 (IO_L4P_0); no longer U$2.127 (IO_L36P_GCLK15_0)
- net A14: now also U$2.134 (IO_L34P_GCLK19_0); no longer U$2.119 (IO_L63P_SCP7_0)
- net A15: now also U$2.137 (IO_L4N_0); no longer U$2.131 (IO_L35N_GCLK16_0)
- net BOUT: now also U$2.117 (IO_L64P_SCP5_0); no longer U$2.94 (IO_L40N_GCLK10_1)
- net CPHI2: now also U$2.94 (IO_L40N_GCLK10_1); no longer U$2.114 (IO_L65N_SCP2_0)
- net GND: now also C72.2, C73.2, C74.2
- net GOUT: now also U$2.119 (IO_L63P_SCP7_0); no longer U$2.95 (IO_L40P_GCLK11_1)
- net GRAPHIC: now also U$2.131 (IO_L35N_GCLK16_0); no longer U$2.137 (IO_L4N_0)
- net HSYNC: now also U$2.115 (IO_L65P_SCP3_0); no longer U$2.99 (IO_L33N_1)
- net IBOUT: now also U$2.116 (IO_L64N_SCP4_0); no longer U$2.93 (IO_L41P_GCLK9_IRDY1_1)
- net IGOUT: no longer U$2.74 (IO_L74N_DOUT_BUSY_1)
- net IROUT: now also U$2.120 (IO_L62N_VREF_0); no longer U$2.105 (IO_L1P_1)
- net PET_VSYNC: now also U$2.105 (IO_L1P_1); no longer U$2.92 (IO_L41N_GCLK8_1)
- net PHI2: now also U$2.99 (IO_L33N_1); no longer U$2.126 (IO_L36N_GCLK14_0)
- net QCLK: now also U$2.95 (IO_L40P_GCLK11_1); no longer U$2.123 (IO_L37N_GCLK12_0)
- net R/-W: now also U$2.97 (IO_L34N_1); no longer U$2.124 (IO_L37P_GCLK13_0)
- net RAMA0: now also U$2.87 (IO_L42N_GCLK6_TRDY1_1); no longer U$2.88 (IO_L42P_GCLK7_1)
- net RAMA1: now also U$2.85 (IO_L43P_GCLK5_1); no longer U$2.87 (IO_L42N_GCLK6_TRDY1_1)
- net RAMA2: now also U$2.84 (IO_L43N_GCLK4_1); no longer U$2.85 (IO_L43P_GCLK5_1)
- net RAMA3: now also U$2.83 (IO_L45P_1); no longer U$2.84 (IO_L43N_GCLK4_1)
- net RAMA4: now also U$2.82 (IO_L45N_1); no longer U$2.83 (IO_L45P_1)
- net RAMD0: now also U$2.80 (IO_L46N_1); no longer U$2.81 (IO_L46P_1)
- net RAMD1: now also U$2.79 (IO_L47P_1); no longer U$2.80 (IO_L46N_1)
- net RAMD2: now also U$2.78 (IO_L47N_1); no longer U$2.79 (IO_L47P_1)
- net RAMD3: now also U$2.75 (IO_L74P_AWAKE_1); no longer U$2.78 (IO_L47N_1)
- net ROUT: no longer U$2.97 (IO_L34N_1)
- net SPI_NAUDIO: now also U$2.127 (IO_L36P_GCLK15_0); no longer U$2.116 (IO_L64N_SCP4_0)
- net SPI_NSEL2: now also U$2.123 (IO_L37N_GCLK12_0)
- net SPI_NSEL3: now also U$2.101 (IO_L32N_1)
- net SPI_NSEL4: now also U$2.124 (IO_L37P_GCLK13_0)
- net V33: now also C72.1, C73.1, C74.1
- net VSYNC: now also U$2.114 (IO_L65N_SCP2_0); no longer U$2.98 (IO_L34P_1)
- net /RAMCS: now also U$2.81 (IO_L46P_1); no longer U$2.82 (IO_L45N_1)
- net /RAMWE: now also U$2.74 (IO_L74N_DOUT_BUSY_1); no longer U$2.75 (IO_L74P_AWAKE_1)
- net /MEMSEL: no longer names the net of U$2.112 (IO_L66P_SCP1_0)
- net SPISELB: no longer names the net of U$2.29 (IO_L36N_3)
- net SPISELC: no longer names the net of U$2.27 (IO_L37P_3)
Other:
- note added: "3.0B: - add pulldown on /RES during FPGA config 3.1A: - replace 5V SRAM with 3.3V SRAM in TSOP2-44 - replace clock oscillator with more common footprint - Change 33R 10kR footprints to SMD - layout-optimized pinout on FPGA - P/N pairs of potential TMDS drivers for vid out - integrated SPI sel demux into FPGA"
- note added: "MICROPET-V3.1A-20250101"
- note removed: "3.0B: - add pulldown on /RES during FPGA config 3.1A: - replace 5V SRAM with 3.3V SRAM in TSOP2-44 - replace clock oscillator with more common footprint - Change 33R 10kR footprints to SMD"
- note removed: "MICROPET-V3.1A-20241230"
