File: Board/I%2fO.kicad_sch (KiCad schematic)
At the start: 33 parts, among them CN3 PORT_CASSETTE_EDGE, CN4 PORT_IEEE_EDGE, IC10 PIAPLCC, IC11 PIAPLCC, IC3 7400D, IC4 7486D, IC5 74145N, IC9 VIAPLCC, P1 C64KEYB, P2 IEEE488FLATCABLE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

Commit message: working on r3.1a
Parts:
- R20, R21: value 10 -> 33; footprint micropet_v3:0207_2V -> Resistor_SMD:R_0805_2012Metric_Pad1.20x1.40mm_HandSolder
Connections:
- net C1MTR: now also CN3.3 (MOTOR), CN3.C (MOTOR@1); no longer CN3.6 (MOTOR), CN3.F (MOTOR@1)
- net C1RD: now also CN3.4 (READ), CN3.D (READ@1); no longer CN3.3 (READ), CN3.C (READ@1)
- net C1SW: now also CN3.6 (SENSE), CN3.F (SENSE@1); no longer CN3.5 (SENSE), CN3.E (SENSE@1)
- net CWR: now also CN3.5 (WRITE), CN3.E (WRITE@1); no longer CN3.4 (WRITE), CN3.D (WRITE@1)
Other:
- note added: "3.0B: - use CPHI2 instead of PHI2 as I/O clock 3.1A: - change 33R footprints to SMD - fix tape PCB edge connector pinout"
- note added: "MICROPET-V3.1A"
- note added: "MICROPET-V3.1A-20241230"
- note removed: "3.0B: - use CPHI2 instead of PHI2 as I/O clock"
- note removed: "MICROPET-V3.0B"
- note removed: "MICROPET-V3.0B-20240523"
Changed lines of the file:
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@@
 	)
 	(junction
-		(at 180.34 274.32)
-		(diameter 0)
-		(color 0 0 0 0)
-	)
-	(junction
 		(at 312.42 139.7)
 		(diameter 0)
@@
 		)
 	)
-	(wire
-		(pts
-			(xy 180.34 274.32) (xy 180.34 269.24)
-		)
-		(stroke
-			(width 0.1524)
-			(type solid)
-		)
-	)
 	(bus
 		(pts
@@
 	(wire
 		(pts
-			(xy 177.8 276.86) (xy 180.34 276.86)
-		)
-		(stroke
-			(width 0.1524)
-			(type solid)
-		)
-	)
-	(wire
-		(pts
 			(xy 261.62 104.14) (xy 261.62 106.68)
 		)
@@
 		)
 	)
-	(wire
-		(pts
-			(xy 185.42 269.24) (xy 185.42 271.78)
-		)
-		(stroke
-			(width 0.1524)
-			(type solid)
-		)
-	)
 	(bus
 		(pts
@@
 	(wire
 		(pts
-			(xy 180.34 269.24) (xy 185.42 269.24)
-		)
-		(stroke
-			(width 0.1524)
-			(type solid)
-		)
-	)
-	(wire
-		(pts
 			(xy 320.04 71.12) (xy 347.98 71.12)
 		)
@@
 		)
 	)
-	(wire
-		(pts
-			(xy 180.34 276.86) (xy 180.34 274.32)
-		)
-		(stroke
-			(width 0.1524)
-			(type solid)
-		)
-	)
 	(polyline
 		(pts
@@
 	(wire
 		(pts
-			(xy 177.8 274.32) (xy 180.34 274.32)
-		)
-		(stroke
-			(width 0.1524)
-			(type solid)
-		)
-	)
-	(wire
-		(pts
 			(xy 127 119.38) (xy 132.08 119.38)
 		)
@@
 		)
 	)
-	(text "MICROPET-V3.0B\n"
+	(text "MICROPET-V3.1A\n"
 		(exclude_from_sim no)
 		(at 452.12 292.1 0)
@@
 		)
 	)
-	(text "MICROPET-V3.0B-20240523"
+	(text "MICROPET-V3.1A-20241230"
 		(exclude_from_sim no)
 		(at 452.12 314.96 0)
@@
 		)
 	)
-	(text "3.0B:\n- use CPHI2 instead of PHI2 as I/O clock"
+	(text "3.0B:\n- use CPHI2 instead of PHI2 as I/O clock\n3.1A:\n- change 33R footprints to SMD\n- fix tape PCB edge connector pinout"
 		(exclude_from_sim no)
-		(at 443.484 277.368 0)
+		(at 445.262 273.304 0)
 		(effects
 			(font
@@
 			)
 		)
-		(property "Value" "10"
+		(property "Value" "33"
 			(at 69.85 206.502 0)
 			(effects
@@
 			)
 		)
-		(property "Footprint" "micropet_v3:0207_2V"
+		(property "Footprint" "Resistor_SMD:R_0805_2012Metric_Pad1.20x1.40mm_HandSolder"
 			(at 73.66 203.2 0)
 			(effects
@@
 	)
 	(symbol
+		(lib_name "PORT_CASSETTE_EDGE_1")
 		(lib_id "micropet_v3-eagle-import:PORT_CASSETTE_EDGE")
 		(at 157.48 289.56 0)
@@
 		(dnp no)
 		(property "Reference" "CN3"
-			(at 157.48 289.56 0)
+			(at 155.956 301.752 0)
 			(effects
 				(font
@@
 		)
 		(property "Footprint" "micropet_v3:MA156_6-2_KEYED"
-			(at 157.48 289.56 0)
+			(at 161.925 275.082 0)
 			(effects
 				(font
@@
 	)
 	(symbol
-		(lib_id "micropet_v3-eagle-import:GND")
-		(at 185.42 274.32 0)
-		(unit 1)
-		(exclude_from_sim no)
-		(in_bom yes)
-		(on_board yes)
-		(dnp no)
-		(property "Reference" "#GND016"
-			(at 185.42 274.32 0)
-			(effects
-				(font
-					(size 1.27 1.27)
-				)
-				(hide yes)
-			)
-		)
-		(property "Value" "GND"
-			(at 182.88 276.86 0)
-			(effects
-				(font
-					(size 1.778 1.5113)
-				)
-				(justify left bottom)
-			)
-		)
-		(property "Footprint" ""
-			(at 185.42 274.32 0)
-			(effects
-				(font
-					(size 1.27 1.27)
-				)
-				(hide yes)
-			)
-		)
-		(property "Datasheet" ""
-			(at 185.42 274.32 0)
-			(effects
-				(font
-					(size 1.27 1.27)
-				)
-				(hide yes)
-			)
-		)
-		(property "Description" ""
-			(at 185.42 274.32 0)
-			(effects
-				(font
-					(size 1.27 1.27)
-				)
-				(hide yes)
-			)
-		)
-		(pin "1"
-		)
-		(instances
-			(project "micropet_v3"
-				(path "/d690d13f-2f18-4476-a6d5-736cfe9a0ec3/40afcc8b-eafe-4576-bdd0-9763391f63cc"
-					(reference "#GND016")
-					(unit 1)
-				)
-			)
-		)
-	)
-	(symbol
 		(lib_id "micropet_v3-eagle-import:RN08")
 		(at 492.76 256.54 180)
@@
 			)
 		)
-		(property "Value" "10"
+		(property "Value" "33"
 			(at 69.85 216.662 0)
 			(effects
@@
 			)
 		)
-		(property "Footprint" "micropet_v3:0207_2V"
+		(property "Footprint" "Resistor_SMD:R_0805_2012Metric_Pad1.20x1.40mm_HandSolder"
 			(at 73.66 213.36 0)
 			(effects
@@
 		(dnp no)
 		(property "Reference" "CN3"
-			(at 121.92 307.34 0)
+			(at 134.112 308.864 0)
 			(effects
 				(font
@@
 		)
 		(property "Footprint" "micropet_v3:MA156_6-2_KEYED"
-			(at 121.92 307.34 0)
+			(at 107.442 302.895 0)
 			(effects
 				(font
