File: Board/Power.kicad_sch (KiCad schematic)
At the start: 79 parts, among them J1 DCJ0202, Q1 IRLML5203, U1 AMS1117-3.3

Commit message: working on r3.1a
Parts:
- R24: footprint micropet_v3:0207_2V -> Resistor_SMD:R_0805_2012Metric_Pad1.20x1.40mm_HandSolder
Other:
- note added: "MICROPET-V3.1A"
- note added: "MICROPET-V3.1A-20241230"
- note added: "V3.0B: - fix footprint for barrel jack power connector V3.1A: - replace THT footprint of 33R with SMD"
- note removed: "MICROPET-V3.0B"
- note removed: "MICROPET-V3.0B-20240505 (MICROPET-V2.1A-20211113)"
- note removed: "V3.0B: - fix footprint for barrel jack power connector"
Changed lines of the file:
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@@
 		)
 	)
-	(text "V3.0B: - fix footprint for barrel jack power connector\n"
+	(text "V3.0B: \n- fix footprint for barrel jack power connector\nV3.1A:\n- replace THT footprint of 33R with SMD\n"
 		(exclude_from_sim no)
-		(at 242.57 164.592 0)
+		(at 218.44 164.084 0)
 		(effects
 			(font
 				(size 2 2)
 			)
+			(justify left)
 		)
 	)
@@
 		)
 	)
-	(text "MICROPET-V3.0B"
+	(text "MICROPET-V3.1A"
 		(exclude_from_sim no)
 		(at 208.28 180.34 0)
@@
 		)
 	)
-	(text "MICROPET-V3.0B-20240505\n(MICROPET-V2.1A-20211113)"
+	(text "MICROPET-V3.1A-20241230"
 		(exclude_from_sim no)
 		(at 244.856 203.454 0)
@@
 			)
 		)
-		(property "Footprint" "micropet_v3:0207_2V"
+		(property "Footprint" "Resistor_SMD:R_0805_2012Metric_Pad1.20x1.40mm_HandSolder"
 			(at 236.22 30.48 0)
 			(effects

Commit message: draft final layout mupet 3.1a
Parts:
- added C75, C76, C77, C78, C79, C80, C81, C82, C83, C84, C85: 0.1u, Capacitor_SMD:C_0603_1608Metric, symbol Device:C_Small
Connections:
- net 3.3V: now also C77.1, C78.1, C79.1, C81.1, C82.1, C83.1, C84.1
- net GND: now also C75.2, C76.2, C77.2, C78.2, C79.2, C80.2, C81.2, C82.2, C83.2, C84.2, C85.2
- net V12: now also C75.1, C76.1, C80.1, C85.1
Other:
- note added: "MICROPET-V3.1A-20250102"
- note added: "U$8"
- note added: "V3.0B: - fix footprint for barrel jack power connector V3.1A: - replace THT footprint of 33R with SMD - add top side bypass caps for FPGA (bottom side bypass caps are optional)"
- note removed: "MICROPET-V3.1A-20241230"
- note removed: "V3.0B: - fix footprint for barrel jack power connector V3.1A: - replace THT footprint of 33R with SMD"
- moved on the sheet: C62, C63, C64, C67, C68, C69

Commit message: usb c connector
Parts:
- removed C26: 47u, micropet_v3:E2,5-6, symbol micropet_v3-eagle-import:CPOL-EUE2.5-6
- removed J1: DCJ0202, micropet_v3:DCJ0202, symbol micropet_v3-eagle-import:DCJ0202
- removed Q1: IRLML5203, micropet_v3:MICRO3, symbol micropet_v3-eagle-import:IRLML5203
- added C26, C86: 47u, micropet_v3:E5-6, symbol micropet_v3-eagle-import:CPOL-EUE5-6
- added J1: USB_C_Receptacle_USB2.0_14P, Connector_USB:USB_C_Receptacle_GCT_USB4085, symbol Connector:USB_C_Receptacle_USB2.0_14P
- added R38: 5k1, micropet_v3:0207_2V, symbol micropet_v3-eagle-import:R-EU_0207/2V
- R16: value 100k -> 5k1
Connections:
- net GND: now also C26.-, C86.-, J1.A1 (GND), J1.A12 (GND), J1.B1 (GND), J1.B12 (GND), J1.S1 (SHIELD), R38.1
- net VCC: now also C26.+, C86.+, J1.A4 (VBUS), J1.A9 (VBUS), J1.B4 (VBUS), J1.B9 (VBUS)
- net at R16.2: now also J1.B5 (CC2)
- new net: J1.A5 (CC1), R38.2
- new net: J1.A6 (D+), J1.B6 (D+)
- new net: J1.A7 (D-), J1.B7 (D-)
Other:
- note added: "MICROPET-V3.1A-20250120"
- note added: "V3.0B: - fix footprint for barrel jack power connector V3.1A: - replace THT footprint of 33R with SMD - add top side bypass caps for FPGA (bottom side bypass caps are optional) - replace barrel power conn with USB-C pwr in"
- note removed: "MICROPET-V3.1A-20250102"
- note removed: "V3.0B: - fix footprint for barrel jack power connector V3.1A: - replace THT footprint of 33R with SMD - add top side bypass caps for FPGA (bottom side bypass caps are optional)"
- moved on the sheet: C5, C6, C7, C8, S1, U1
