File: Board/micropet_v3.kicad_pcb (KiCad board)
At the start: 2 copper layers, 190.2 x 100.3 mm, 183 parts, among them CN3 PORT_CASSETTE_EDGE, CN4 PORT_IEEE_EDGE, IC1 RAMSOCK32TO512KSOP, IC10 PIAPLCC, IC11 PIAPLCC, IC13 RAMSOCK32TO512KSOP, IC16 74LVC8T245SO24, IC2 74245DW, IC3 7400D, IC4 7486D, IC5 74145N, IC6 74125D, IC7 74138D, IC8 MAX3421E, IC9 VIAPLCC, J1 DCJ0202, P1 C64KEYB, P2 IEEE488FLATCABLE, P3 PETUSERPORT, P6 CBMTAPE, P7 PETKEYBD, Q1 IRLML5203, Q2 32kHz, Q3 12MHz, U1 AMS1117-3.3, U2 74LVC1G04, X1 1503_09, X2 D-SUB15-HDR15RA

Commit message: working on r3.1a
Parts:
- removed JS1: RENOSCXLH, micropet_v3:RENJS6
- added R33: 10k, Resistor_SMD:R_0805_2012Metric_Pad1.20x1.40mm_HandSolder, F.Cu at (60.5, 88.2)
- added R34: 10k, Resistor_SMD:R_0805_2012Metric_Pad1.20x1.40mm_HandSolder, F.Cu at (68.0, 83.5)
- added R35: 10k, Resistor_SMD:R_0805_2012Metric_Pad1.20x1.40mm_HandSolder, F.Cu at (68.0, 86.5)
- added R36: 4k7, micropet_v3:0204V, F.Cu at (75.4, 27.5)
- added R37: 470, micropet_v3:0204V, F.Cu at (75.4, 30.4)
- added X3: SG-8002CE, Oscillator:Oscillator_SMD_SeikoEpson_SG8002CE-4Pin_3.2x2.5mm, F.Cu at (60.9, 84.4)
- IC1, IC13: value RAMSOCK32TO512KSOP -> 512k x8 10ns SRAM; footprint micropet_v3:SOP32 -> Package_SO:TSOP-II-44_10.16x18.41mm_P0.8mm
- IC8: footprint micropet_v3:TQFP32-5MM -> Package_QFP:LQFP-32_5x5mm_P0.5mm
- R1, R2, R4: footprint micropet_v3:0204_7 -> Resistor_SMD:R_0805_2012Metric_Pad1.20x1.40mm_HandSolder
- R10, R11, R24, R9: footprint micropet_v3:0207_2V -> Resistor_SMD:R_0805_2012Metric_Pad1.20x1.40mm_HandSolder
- R12: value 3k3 -> 4k7
- R20, R21: value 10 -> 33; footprint micropet_v3:0207_2V -> Resistor_SMD:R_0805_2012Metric_Pad1.20x1.40mm_HandSolder
Connections:
- C52 pad 1: Net-(C49-Pad1) -> Net-(C52-Pad1)
- CN3 pad 3: /I/O/C1RD -> /I/O/C1MTR
- CN3 pad 4: /I/O/CWR -> /I/O/C1RD
- CN3 pad 5: /I/O/C1SW -> /I/O/CWR
- CN3 pad 6: /I/O/C1MTR -> /I/O/C1SW
- CN3 pad C: /I/O/C1RD -> /I/O/C1MTR
- CN3 pad D: /I/O/CWR -> /I/O/C1RD
- CN3 pad E: /I/O/C1SW -> /I/O/CWR
- CN3 pad F: /I/O/C1MTR -> /I/O/C1SW
- IC1 pad 1: /CPU,RAM,ROM/FA18 -> unconnected-(IC1-NC-Pad1)
- IC1 pad 10: A2 -> D1
- IC1 pad 11: A1 -> V33
- IC1 pad 12: A0 -> GND
- IC1 pad 13: D0 -> D2
- IC1 pad 14: D1 -> D3
- IC1 pad 15: D2 -> R/-W
- IC1 pad 16: GND -> A5
- IC1 pad 17: D3 -> A6
- IC1 pad 18: D4 -> A7
- IC1 pad 19: D5 -> A8
- IC1 pad 2: /CPU,RAM,ROM/FA16 -> unconnected-(IC1-NC-Pad2)
- IC1 pad 20: D6 -> A9
- IC1 pad 21: D7 -> unconnected-(IC1-NC-Pad21)
- IC1 pad 22: /CPU,RAM,ROM//FRAMSEL -> unconnected-(IC1-NC-Pad22)
- IC1 pad 23: /CPU,RAM,ROM/A10 -> unconnected-(IC1-NC-Pad23)
- IC1 pad 24: /CPU,RAM,ROM//FRAMSEL -> unconnected-(IC1-NC-Pad24)
- IC1 pad 25: /CPU,RAM,ROM/A11 -> unconnected-(IC1-NC-Pad25)
- IC1 pad 26: /CPU,RAM,ROM/A9 -> A10
- IC1 pad 27: /CPU,RAM,ROM/A8 -> A11
- IC1 pad 28: /CPU,RAM,ROM/A13 -> A12
- IC1 pad 29: R/-W -> A13
- IC1 pad 3: /CPU,RAM,ROM/A14 -> A0
- IC1 pad 30: /CPU,RAM,ROM/FA17 -> A14
- IC1 pad 31: /CPU,RAM,ROM/FA15 -> D4
- IC1 pad 32: V33 -> D5
- IC1 pad 4: /CPU,RAM,ROM/A12 -> A1
- IC1 pad 5: /CPU,RAM,ROM/A7 -> A2
- IC1 pad 6: /CPU,RAM,ROM/A6 -> A3
- IC1 pad 7: /CPU,RAM,ROM/A5 -> A4
- IC1 pad 8: /CPU,RAM,ROM/A4 -> /CPU,RAM,ROM//FRAMSEL
- IC1 pad 9: A3 -> D0
- IC13 pad 1: /CPU,RAM,ROM/RAMA18 -> unconnected-(IC13-NC-Pad1)
- IC13 pad 10: /CPU,RAM,ROM/RAMA2 -> RAMD1
- IC13 pad 11: /CPU,RAM,ROM/RAMA1 -> V33
- IC13 pad 12: /CPU,RAM,ROM/RAMA0 -> GND
- IC13 pad 13: /CPU,RAM,ROM/RAMD0 -> RAMD2
- IC13 pad 14: /CPU,RAM,ROM/RAMD1 -> RAMD3
- IC13 pad 15: /CPU,RAM,ROM/RAMD2 -> /RAMWE
- IC13 pad 16: GND -> RAMA5
- IC13 pad 17: /CPU,RAM,ROM/RAMD3 -> RAMA6
- IC13 pad 18: /CPU,RAM,ROM/RAMD4 -> RAMA7
- IC13 pad 19: /CPU,RAM,ROM/RAMD5 -> RAMA8
- IC13 pad 2: /CPU,RAM,ROM/RAMA16 -> unconnected-(IC13-NC-Pad2)
- IC13 pad 20: /CPU,RAM,ROM/RAMD6 -> RAMA9
- IC13 pad 21: /CPU,RAM,ROM/RAMD7 -> unconnected-(IC13-NC-Pad21)
- IC13 pad 22: /CPU,RAM,ROM//RAMCS -> unconnected-(IC13-NC-Pad22)
- IC13 pad 23: /CPU,RAM,ROM/RAMA10 -> unconnected-(IC13-NC-Pad23)
- IC13 pad 24: /CPU,RAM,ROM//RAMCS -> unconnected-(IC13-NC-Pad24)
- IC13 pad 25: /CPU,RAM,ROM/RAMA11 -> unconnected-(IC13-NC-Pad25)
- IC13 pad 26: /CPU,RAM,ROM/RAMA9 -> RAMA10
- IC13 pad 27: /CPU,RAM,ROM/RAMA8 -> RAMA11
- IC13 pad 28: /CPU,RAM,ROM/RAMA13 -> RAMA12
- IC13 pad 29: /CPU,RAM,ROM//RAMWE -> RAMA13
- IC13 pad 3: /CPU,RAM,ROM/RAMA14 -> RAMA0
- IC13 pad 30: /CPU,RAM,ROM/RAMA17 -> RAMA14
- IC13 pad 31: /CPU,RAM,ROM/RAMA15 -> RAMD4
- IC13 pad 32: V33 -> RAMD5
- IC13 pad 4: /CPU,RAM,ROM/RAMA12 -> RAMA1
- IC13 pad 5: /CPU,RAM,ROM/RAMA7 -> RAMA2
- IC13 pad 6: /CPU,RAM,ROM/RAMA6 -> RAMA3
- IC13 pad 7: /CPU,RAM,ROM/RAMA5 -> RAMA4
- IC13 pad 8: /CPU,RAM,ROM/RAMA4 -> /RAMCS
- IC13 pad 9: /CPU,RAM,ROM/RAMA3 -> RAMD0
- IC6 pad 3: /CPU,RAM,ROM/RAMA3 -> RAMA5
- IC6 pad 6: /CPU,RAM,ROM/FA18 -> FA18
- IC8 pad 1: unconnected-(IC8-GPIN7-Pad1) -> Net-(IC8-GPIN7)
- IC8 pad 32: unconnected-(IC8-GPIN6-Pad32) -> Net-(IC8-GPIN6)
- U$1 pad 15: /CPU,RAM,ROM/A4 -> A4
- U$1 pad 16: /CPU,RAM,ROM/A5 -> A5
- U$1 pad 17: /CPU,RAM,ROM/A6 -> A6
- U$1 pad 18: /CPU,RAM,ROM/A7 -> A7
- U$1 pad 19: /CPU,RAM,ROM/A8 -> A8
- U$1 pad 20: /CPU,RAM,ROM/A9 -> A9
- U$1 pad 21: /CPU,RAM,ROM/A10 -> A10
- U$1 pad 22: /CPU,RAM,ROM/A11 -> A11
- U$1 pad 25: /CPU,RAM,ROM/A12 -> A12
- U$1 pad 26: /CPU,RAM,ROM/A13 -> A13
- U$1 pad 27: /CPU,RAM,ROM/A14 -> A14
- U$2 pad 10: /CPU,RAM,ROM/A9 -> A9
- U$2 pad 11: /CPU,RAM,ROM/A10 -> A10
- U$2 pad 119: /CPU,RAM,ROM/A14 -> A14
- U$2 pad 127: /CPU,RAM,ROM/A12 -> A12
- U$2 pad 139: /CPU,RAM,ROM/A13 -> A13
- U$2 pad 140: /CPU,RAM,ROM/FA15 -> FA15
- U$2 pad 141: /CPU,RAM,ROM/FA16 -> FA16
- U$2 pad 142: /CPU,RAM,ROM/A11 -> A11
- U$2 pad 143: /CPU,RAM,ROM/FA17 -> FA17
- U$2 pad 144: /CPU,RAM,ROM/FA18 -> FA18
- U$2 pad 26: /CPU,RAM,ROM/A7 -> A7
- U$2 pad 30: /CPU,RAM,ROM/A8 -> A8
- U$2 pad 33: /CPU,RAM,ROM/A6 -> A6
- U$2 pad 35: /CPU,RAM,ROM/A4 -> A4
- U$2 pad 40: /CPU,RAM,ROM/A5 -> A5
- U$2 pad 43: /CPU,RAM,ROM/RAMD3 -> RAMA14
- U$2 pad 44: /CPU,RAM,ROM/RAMD2 -> RAMA13
- U$2 pad 45: /CPU,RAM,ROM/RAMD4 -> RAMA12
- U$2 pad 46: /CPU,RAM,ROM/RAMD1 -> RAMA11
- U$2 pad 47: /CPU,RAM,ROM/RAMD5 -> RAMA10
- U$2 pad 48: /CPU,RAM,ROM/RAMD0 -> RAMD4
- U$2 pad 50: /CPU,RAM,ROM/RAMD6 -> RAMD5
- U$2 pad 51: /CPU,RAM,ROM/RAMA0 -> RAMD6
- U$2 pad 55: /CPU,RAM,ROM/RAMD7 -> RAMD7
- U$2 pad 56: /CPU,RAM,ROM/RAMA1 -> RAMA15
- U$2 pad 57: /CPU,RAM,ROM/RAMA10 -> RAMA16
- U$2 pad 58: /CPU,RAM,ROM/RAMA2 -> RAMA17
- U$2 pad 59: /CPU,RAM,ROM//RAMCS -> RAMA18
- U$2 pad 60: /CPU,RAM,ROM/RAMA3 -> RAMA5
- U$2 pad 61: /CPU,RAM,ROM/RAMA4 -> RAMA6
- U$2 pad 62: /CPU,RAM,ROM/RAMA11 -> RAMA7
- U$2 pad 66: /CPU,RAM,ROM/RAMA5 -> RAMA8
- U$2 pad 69: /CPU,RAM,ROM/RAMA9 -> RAMA9
- U$2 pad 75: /CPU,RAM,ROM/RAMA6 -> /RAMWE
- U$2 pad 78: /CPU,RAM,ROM/RAMA8 -> RAMD3
- U$2 pad 79: /CPU,RAM,ROM/RAMA7 -> RAMD2
- U$2 pad 80: /CPU,RAM,ROM/RAMA13 -> RAMD1
- U$2 pad 81: /CPU,RAM,ROM/RAMA12 -> RAMD0
- U$2 pad 82: /CPU,RAM,ROM//RAMWE -> /RAMCS
- U$2 pad 83: /CPU,RAM,ROM/RAMA14 -> RAMA4
- U$2 pad 84: /CPU,RAM,ROM/RAMA17 -> RAMA3
- U$2 pad 85: /CPU,RAM,ROM/RAMA16 -> RAMA2
- U$2 pad 87: /CPU,RAM,ROM/RAMA15 -> RAMA1
- U$2 pad 88: /CPU,RAM,ROM/RAMA18 -> RAMA0
Routing:
- net (no net): track 0.00 -> 209.2 mm, vias 0 -> 14
- net /CPU,RAM,ROM/A14: track 82.5 -> 0.00 mm, vias 7 -> 0
- net RAMA5: track 0.00 -> 79.4 mm, vias 0 -> 2
- net FA18: track 0.00 -> 76.7 mm, vias 0 -> 3
- net /CPU,RAM,ROM/FA18: track 76.7 -> 0.00 mm, vias 3 -> 0
- net /CPU,RAM,ROM/RAMA3: track 73.3 -> 0.00 mm, vias 2 -> 0
- net A13: track 0.00 -> 73.2 mm, vias 0 -> 3
- net /CPU,RAM,ROM/A13: track 73.2 -> 0.00 mm, vias 3 -> 0
- net /CPU,RAM,ROM/A12: track 68.3 -> 0.00 mm, vias 5 -> 0
- net /CPU,RAM,ROM/FA17: track 58.5 -> 0.00 mm, vias 2 -> 0
- net A11: track 0.00 -> 57.4 mm, vias 0 -> 3
- net /CPU,RAM,ROM/A11: track 57.4 -> 0.00 mm, vias 3 -> 0
- net FA15: track 0.00 -> 56.6 mm, vias 0 -> 2
- net /CPU,RAM,ROM/FA15: track 56.6 -> 0.00 mm, vias 2 -> 0
- net A10: track 0.00 -> 49.8 mm, vias 0 -> 1
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
Commit message: draft final layout mupet 3.1a
Parts:
- removed IC7: 74138D, micropet_v3:SO16
- added C72: 0.1u, Capacitor_SMD:C_0603_1608Metric, F.Cu at (91.5, 77.5)
- added C73: 0.1u, Capacitor_SMD:C_0603_1608Metric, F.Cu at (92.8, 94.2)
- added C74: 0.1u, Capacitor_SMD:C_0603_1608Metric, F.Cu at (91.8, 106.0)
- added C75: 0.1u, Capacitor_SMD:C_0603_1608Metric, F.Cu at (102.6, 107.3)
- added C76: 0.1u, Capacitor_SMD:C_0603_1608Metric, F.Cu at (116.8, 124.6)
- added C77: 0.1u, Capacitor_SMD:C_0603_1608Metric, F.Cu at (119.1, 124.6)
- added C78: 0.1u, Capacitor_SMD:C_0603_1608Metric, F.Cu at (113.3, 123.7)
- added C79: 0.1u, Capacitor_SMD:C_0603_1608Metric, F.Cu at (102.6, 108.8)
- added C80: 0.1u, Capacitor_SMD:C_0603_1608Metric, F.Cu at (111.6, 94.5)
- added C81: 0.1u, Capacitor_SMD:C_0603_1608Metric, F.Cu at (104.9, 119.3)
- added C82: 0.1u, Capacitor_SMD:C_0603_1608Metric, F.Cu at (132.8, 104.6)
- added C83: 0.1u, Capacitor_SMD:C_0603_1608Metric, F.Cu at (124.6, 94.5)
- added C84: 0.1u, Capacitor_SMD:C_0603_1608Metric, F.Cu at (116.6, 94.5)
- added C85: 0.1u, Capacitor_SMD:C_0603_1608Metric, F.Cu at (132.8, 106.3)
- added JP11: JP1E, micropet_v3:JP1, F.Cu at (102.1, 70.5)
- added JP12: JP1E, micropet_v3:JP1, F.Cu at (98.6, 70.5)
- moved X3 85.7 mm to (132.8, 131.1)
- moved R33 80.3 mm to (128.5, 131.0), turned to -90 degrees
- moved R34 49.1 mm to (113.2, 64.5), turned to 180 degrees
- moved R35 49.1 mm to (113.2, 67.5), turned to 180 degrees
- moved R37 21.8 mm to (84.0, 50.5)
- moved R36 21.8 mm to (84.0, 47.5)
- moved C13 1.65 mm to (129.8, 134.2), turned to 0 degrees
- moved R24 1.07 mm to (144.2, 136.0)
Connections:
- U$2 pad 101: unconnected-(U$2A-IO_L32N_1-Pad101) -> SPI_NSEL3
- U$2 pad 102: /CPU,RAM,ROM/C8PHI2 -> /CPU,RAM,ROM/SPI_NFLASH
- U$2 pad 104: /CPU,RAM,ROM/C2PHI2 -> SPI_NSEL5
- U$2 pad 105: IROUT -> PET_VSYNC
- U$2 pad 111: /SEL4 -> unconnected-(U$2A-IO_L66N_SCP0_0-Pad111)
- U$2 pad 112: /CPU,RAM,ROM//MEMSEL -> unconnected-(U$2A-IO_L66P_SCP1_0-Pad112)
- U$2 pad 114: CPHI2 -> VSYNC
- U$2 pad 115: /SEL2 -> HSYNC
- U$2 pad 116: SPI_NAUDIO -> IBOUT
- U$2 pad 117: /RES -> BOUT
- U$2 pad 118: /CPU,RAM,ROM/BE_IN -> IGOUT
- U$2 pad 119: A14 -> GOUT
- U$2 pad 120: /CPU,RAM,ROM//FRAMSEL -> IROUT
- U$2 pad 121: /CPU,RAM,ROM/SYNC -> ROUT
- U$2 pad 123: /CPU,RAM,ROM/QCLK -> SPI_NSEL2
- U$2 pad 124: R/-W -> SPI_NSEL4
- U$2 pad 126: PHI2 -> /LDAC
- U$2 pad 127: A12 -> SPI_NAUDIO
- U$2 pad 131: /CPU,RAM,ROM/A15 -> GRAPHIC
- U$2 pad 132: /CPU,RAM,ROM//BE_OUT -> /CPU,RAM,ROM//FRAMSEL
- U$2 pad 134: /SEL1 -> A14
- U$2 pad 137: GRAPHIC -> /CPU,RAM,ROM/A15
- U$2 pad 138: /LDAC -> A12
- U$2 pad 27: /CPU,RAM,ROM/SPISELC -> unconnected-(U$2A-IO_L37P_3-Pad27)
- U$2 pad 29: /CPU,RAM,ROM/SPISELB -> unconnected-(U$2A-IO_L36N_3-Pad29)
- U$2 pad 38: /CPU,RAM,ROM/SPISELA -> /CPU,RAM,ROM//FPGABOOT
- U$2 pad 74: IGOUT -> /RAMWE
- U$2 pad 75: /RAMWE -> RAMD3
- U$2 pad 78: RAMD3 -> RAMD2
- U$2 pad 79: RAMD2 -> RAMD1
- U$2 pad 80: RAMD1 -> RAMD0
- U$2 pad 81: RAMD0 -> /RAMCS
- U$2 pad 82: /RAMCS -> RAMA4
- U$2 pad 83: RAMA4 -> RAMA3
- U$2 pad 84: RAMA3 -> RAMA2
- U$2 pad 85: RAMA2 -> RAMA1
- U$2 pad 87: RAMA1 -> RAMA0
- U$2 pad 88: RAMA0 -> /SEL4
- U$2 pad 92: PET_VSYNC -> /SEL2
- U$2 pad 93: IBOUT -> /SEL1
- U$2 pad 94: BOUT -> CPHI2
- U$2 pad 95: GOUT -> /CPU,RAM,ROM/QCLK
- U$2 pad 97: ROUT -> R/-W
- U$2 pad 98: VSYNC -> /RES
- U$2 pad 99: HSYNC -> PHI2
Routing:
- net (no net): track 209.2 -> 0.00 mm, vias 14 -> 0
- net GND: track 1982.0 -> 2164.3 mm, vias 104 -> 121
- net A14: track 0.00 -> 71.3 mm, vias 0 -> 6
- net FA17: track 0.00 -> 67.1 mm, vias 0 -> 4
- net A12: track 0.00 -> 65.8 mm, vias 0 -> 5
- net V33: track 802.2 -> 864.6 mm, vias 54 -> 60
- net /CPU,RAM,ROM/SPISELA: track 61.0 -> 0.00 mm, vias 2 -> 0
- net /CPU,RAM,ROM/SPISELC: track 56.8 -> 0.00 mm, vias 2 -> 0
- net /CPU,RAM,ROM/SPISELB: track 55.2 -> 0.00 mm, vias 2 -> 0
- net SPI_NSEL3: track 125.5 -> 85.0 mm, vias 2 -> 4
- net /CPU,RAM,ROM//FPGABOOT: track 83.6 -> 43.2 mm, vias 5 -> 2
- net /CPU,RAM,ROM/SPI_NFLASH: track 49.9 -> 15.6 mm, vias 3 -> 0
- net Net-(IC8-GPIN7): track 0.00 -> 34.1 mm, vias 0 -> 2
- net D5: track 110.5 -> 77.2 mm, vias 7 -> 6
- net Net-(IC8-GPIN6): track 0.00 -> 32.3 mm, vias 0 -> 2
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Other:
- board text added: "(C) 2025 A. Fachat"
- board text added: "/RES on IEEE488"
- board text added: "6521 PIA"
- board text added: "6522 VIA"
- board text added: "JP10: 1-2: ATNA 2-3: orig U$8: USB-C Pwr in (adafr.)"
- board text added: "JP11/12: boot opt"
- board text added: "JP6: 1-2: orig 2-3: ATNIN"
- board text added: "JP9: VCC on UP Video"
- board text added: "KBD extra"
- board text added: "MicroPET-V3.1A"
- board text added: "PWR LED"
- board text added: "TTL C1MTR"
- board text added: "TTL C2MTR"
- board text added: "Tape 2"
- board text added: "Trigger FPGA Config"
- board text added: "X1"
- board text removed: "MicroPET-V3.0B"

Commit message: usb c connector
Parts:
- removed Q1: IRLML5203, micropet_v3:MICRO3
- added C86: 47u, micropet_v3:E5-6, F.Cu at (85.6, 73.5)
- added R38: 5k1, micropet_v3:0207_2V, F.Cu at (257.6, 53.7)
- C26: footprint micropet_v3:E2,5-6 -> micropet_v3:E5-6
- J1: value DCJ0202 -> USB_C_Receptacle_USB2.0_14P; footprint micropet_v3:DCJ0202 -> Connector_USB:USB_C_Receptacle_GCT_USB4085
- R16: value 100k -> 5k1
- moved C26 102.3 mm to (256.9, 71.3), turned to 0 degrees
- moved C14 3.49 mm to (89.7, 70.2)
- moved J1 2.93 mm to (253.7, 65.2)
- moved R16 2.01 mm to (260.6, 53.7), turned to -90 degrees
- moved R29 1.02 mm to (111.3, 127.4)
Connections:
- R16 pad 2: Net-(Q1-G) -> Net-(J1-CC2)
Routing:
- net VCC: track 997.4 -> 1135.1 mm, vias 37 -> 42
- net V33: track 864.6 -> 881.6 mm, vias 60 -> 62
- net Net-(J1-CC1): track 0.00 -> 15.0 mm
- net Net-(J1-CC2): track 0.00 -> 10.5 mm
- net Net-(Q1-D): track 10.4 -> 0.00 mm
- net GND: track 2164.3 -> 2155.5 mm, vias 121 -> 120
- net Net-(Q1-G): track 4.35 -> 0.00 mm
- net SPI_MISO: track 198.7 -> 194.5 mm
- net SPI_CLK: track 201.6 -> 199.1 mm
- net Net-(J1-D+-PadA6): track 0.00 -> 1.99 mm
- net Net-(J1-D--PadA7): track 0.00 -> 1.93 mm
- net SPI_MOSI: track 206.3 -> 204.7 mm
- net /USB/DETECT: track 47.2 -> 48.4 mm
- net SPI_IN3: track 69.5 -> 70.8 mm
- net /CPU,RAM,ROM/DONE: track 74.1 -> 73.4 mm
Other:
- board text added: "JP10: 1-2: ATNA 2-3: orig"
- board text added: "U$8: USB-C Pwr in (adafr.)"
- board text removed: "JP10: 1-2: ATNA 2-3: orig U$8: USB-C Pwr in (adafr.)"
