File: Board/USB.kicad_sch (KiCad schematic)
At the start: 22 parts, among them IC8 MAX3421E, Q2 32kHz, Q3 12MHz

Commit message: working on r3.1a
Parts:
- added JP11, JP12: JP1E, csa_ultracpu:JP1, symbol csa_ultracpu-eagle-import:JP1E
- added R34, R35: 10k, Resistor_SMD:R_0805_2012Metric_Pad1.20x1.40mm_HandSolder, symbol csa_ultracpu-eagle-import:R-EU_0204/7
- IC8: footprint micropet_v3:TQFP32-5MM -> Package_QFP:LQFP-32_5x5mm_P0.5mm
- R1, R2, R4: footprint micropet_v3:0204_7 -> Resistor_SMD:R_0805_2012Metric_Pad1.20x1.40mm_HandSolder
Connections:
- net 3.3V: now also R34.2, R35.2
- net GND: now also JP11.1, JP12.1
- net at IC8.1 (GPIN7): now also JP12.2, R35.1
- net at IC8.32 (GPIN6): now also JP11.2, R34.1
Other:
- note added: "3.1A: - replace THT footprints for 33R with SMD - replace non-commercial MAX3421 footprint with kicad one - add boot option jumpsd on USB GPIN"
- note added: "MICROPET-V3.1A"
- note added: "MICROPET-V3.1A-20241230"
- note removed: "MICROPET-V2.0A-20210306"
- note removed: "MICROPET-V3.0A"
- note removed: "Non-commercial use only"
- note removed: "Note: MAX3421 TQFP-5MM"
- note removed: "Note: Micro-USB package"
- note removed: "package layout by SparkFun"

Commit message: draft final layout mupet 3.1a
Parts:
- JP11, JP12: footprint csa_ultracpu:JP1 -> micropet_v3:JP1
Changed lines of the file:
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@@
 			)
 		)
-		(property "Footprint" "csa_ultracpu:JP1"
+		(property "Footprint" "micropet_v3:JP1"
 			(at 45.72 139.7 0)
 			(effects
@@
 			)
 		)
-		(property "Footprint" "csa_ultracpu:JP1"
+		(property "Footprint" "micropet_v3:JP1"
 			(at 45.72 132.08 0)
 			(effects

Commit message: final touches, 22u audio output caps
Other:
- note added: "3.1A: - replace THT footprints for 33R with SMD - replace non-commercial MAX3421 footprint with kicad one - add boot option jumper on USB GPIN"
- note removed: "3.1A: - replace THT footprints for 33R with SMD - replace non-commercial MAX3421 footprint with kicad one - add boot option jumpsd on USB GPIN"
Changed lines of the file:
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@@
 		)
 	)
-	(text "3.1A:\n- replace THT footprints for 33R with SMD\n- replace non-commercial MAX3421 footprint with kicad one\n- add boot option jumpsd on USB GPIN"
+	(text "3.1A:\n- replace THT footprints for 33R with SMD\n- replace non-commercial MAX3421 footprint with kicad one\n- add boot option jumper on USB GPIN"
 		(exclude_from_sim no)
 		(at 99.314 188.214 0)
